Commit message: add conveyor

File: urdf/conveyor.urdf (robot description, URDF)
Before this commit: robot liukuhihna_gazebo, 3 links, 2 joints
Links:
- link belt_visual: geometry collision mesh filename=package://panda_moveit_config/meshes/conveyor_simple.stl; visual mesh filename=package://panda_moveit_config/meshes/conveyor_belt.stl
