Commit message: Change box size; change spawn frequency.

File: urdf/box.urdf (robot description, URDF)
Before this commit: robot box, 1 links, 0 joints
Links:
- link base_link: mass 0.05 -> 0.5; geometry collision box size=0.5 0.1 0.2; visual box size=0.5 0.1 0.2

Commit message: modify script

File: urdf/box.urdf (robot description, URDF)
Before this commit: robot box, 1 links, 0 joints
Links:
- link base_link: mass 0.5 -> 0.1

Commit message: modify gazebo

File: urdf/box.urdf (robot description, URDF)
Before this commit: robot box, 1 links, 0 joints
Links:
- link base_link: geometry collision box size=0.5 0.1 0.25; visual box size=0.5 0.1 0.25

File: urdf/red_cylinder.urdf (robot description, URDF)
Before this commit: robot red_cylinder, 1 links, 0 joints
Links:
- link base_link: mass 0.01 -> 0.01100001
